Commit message: v4 initial firmware

File: packages/main/config/robot.urdf (robot description, URDF)
Before this commit: robot my_robot, 2 links, 1 joints
Links:
- added link tof_lidar
Joints:
- added joint tof_lidar_joint: type fixed, parent base_link, child tof_lidar, origin xyz=0.09 0 -0.08 rpy=-1.57 0 -1.57
- joint lidar_joint: origin xyz=0.06 0 0 rpy=0 0 1.57 -> xyz=0.06 0 0 rpy=0 0 0
